Commit message: fix transforms in urdf, publish frameid in imucalib

File: SAILMAV.urdf (robot description, URDF)
Before this commit: robot SAILMAV, 4 links, 4 joints
Links:
- removed link camera_link
- added link right_camera_link; visual box size=0.06 0.04 0.02
Joints:
- removed joint camera_joint
- joint left_camera_joint: origin xyz=0 0.19 0 rpy=-1.57 0 -1.57 -> xyz=0 0.19 0 rpy=-3.14 0 -1.57
- joint right_camera_joint: child left_camera_link -> right_camera_link; origin xyz=0 -0.19 0 rpy=-1.57 0 -1.57 -> xyz=0 -0.19 0 rpy=-3.14 0 -1.57

Commit message: fix urdf, update a param

File: SAILMAV.urdf (robot description, URDF)
Before this commit: robot SAILMAV, 4 links, 4 joints
Links:
- removed link camera_link
- added link right_camera_link; visual box size=0.06 0.04 0.02
Joints:
- removed joint camera_joint
- joint right_camera_joint: child left_camera_link -> right_camera_link
